File: projects/TempHumiSensor/esp8266_01.sch (EAGLE design)
At the start: 14 parts

Commit message: layout
Parts:
- removed R6: 4.7k, SparkFun-Resistors:RESISTOR0805-RES
Connections:
- removed net N$6: R6.1
- net 3.3V: no longer R6.2
Changed lines of the file:
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@@
 <?xml version="1.0" encoding="utf-8"?>
 <!DOCTYPE eagle SYSTEM "eagle.dtd">
-<eagle version="7.2.0">
+<eagle version="7.5.0">
 <drawing>
 <settings>
@@
 <classes>
 <class number="0" name="default" width="0.508" drill="0.254">
-<clearance class="0" value="0.508"/>
+<clearance class="0" value="0.254"/>
 </class>
 </classes>
@@
 <part name="R4" library="SparkFun-Resistors" deviceset="RESISTOR" device="0805-RES" value="4.7k"/>
 <part name="R5" library="SparkFun-Resistors" deviceset="RESISTOR" device="0805-RES" value="4.7k"/>
-<part name="R6" library="SparkFun-Resistors" deviceset="RESISTOR" device="0805-RES" value="4.7k"/>
 <part name="SUPPLY3" library="SparkFun-Aesthetics" deviceset="3.3V" device=""/>
 <part name="CN1" library="adafruit" deviceset="DCBARREL" device="PTH"/>
@@
 <instance part="R4" gate="G$1" x="50.8" y="71.12" rot="R90"/>
 <instance part="R5" gate="G$1" x="58.42" y="71.12" rot="R90"/>
-<instance part="R6" gate="G$1" x="66.04" y="71.12" rot="R90"/>
 <instance part="SUPPLY3" gate="G$1" x="50.8" y="78.74"/>
 <instance part="CN1" gate="G$1" x="-20.32" y="63.5"/>
@@
 <pinref part="R5" gate="G$1" pin="2"/>
 <wire x1="50.8" y1="76.2" x2="58.42" y2="76.2" width="0.1524" layer="91"/>
-<pinref part="R6" gate="G$1" pin="2"/>
-<wire x1="58.42" y1="76.2" x2="66.04" y2="76.2" width="0.1524" layer="91"/>
 <label x="45.72" y="76.2" size="1.778" layer="95"/>
 <pinref part="SUPPLY3" gate="G$1" pin="3.3V"/>
@@
 </segment>
 </net>
-<net name="N$6" class="0">
-<segment>
-<pinref part="R6" gate="G$1" pin="1"/>
-<wire x1="66.04" y1="66.04" x2="66.04" y2="58.42" width="0.1524" layer="91"/>
-<label x="66.04" y="58.42" size="1.778" layer="95" rot="R90"/>
-</segment>
-</net>
